Commit message: simple_fix_location

File: src/ugv_sim/scout_description/urdf/laser.xacro (robot description, xacro)
@@ -3,6 +3,6 @@
     <joint name="chassis_front_laser_joint" type="fixed">
         <axis xyz="0 0 1"/>
-        <origin rpy="0 0 0" xyz="0 0.0 0.16"/>
-        <parent link="base_link"/>
+        <origin rpy="0 0 0" xyz="0 0 0.1"/>
+        <parent link="velodyne_base_link"/>
         <child link="front_laser"/>
     </joint>
