Commit message: update_depth_camera.xacro

File: src/ugv_sim/scout_description/urdf/camera.xacro (robot description, xacro)
@@ -1,55 +1,54 @@
 <?xml version="1.0"?>
 <robot xmlns:xacro="http://www.ros.org/wiki/xacro">
-    <!-- 카메라 링크 추가 -->
-    <joint name="camera_mount_joint" type="fixed">
-        <origin rpy="0 0 0" xyz="0.2 0 0.057"/>
-        <parent link="base_link"/>
-        <child link="camera_link"/>
-    </joint>
-    <link name="camera_link">
-        <inertial>
-            <mass value="0.1"/>
-            <origin xyz="0 0 0"/>
-            <inertia ixx="0.001" ixy="0" ixz="0" iyy="0.001" iyz="0" izz="0.001"/>
-        </inertial>
-        <visual>
-            <geometry>
-                <box size="0.02 0.04 0.01"/>
-            </geometry>
-            <material name="white">
-                <color rgba="0.1 0.1 0.8 1.0"/>
-            </material>
-        </visual>
-        <collision>
-            <geometry>
-                <box size="0.05 0.05 0.05"/>
-            </geometry>
-        </collision>
-    </link>
-    <!-- 컬러 카메라 센서 -->
-    <gazebo reference="camera_link">
-        <sensor name="color_camera" type="camera">
-            <camera>
-                <horizontal_fov>1.3962634</horizontal_fov>
-                <image>
-                    <width>640</width>
-                    <height>480</height>
-                    <format>R8G8B8</format>
-                </image>
-                <clip>
-                    <near>0.1</near>
-                    <far>10</far>
-                </clip>
-            </camera>
-            <always_on>true</always_on>
-            <update_rate>30</update_rate>
-            <visualize>true</visualize>
-            <plugin name="color_camera_controller" filename="libgazebo_ros_camera.so">
-            <camera_name>camera</camera_name>
-            <image_topic_name>image_raw</image_topic_name>
-            <camera_info_topic_name>camera_info</camera_info_topic_name>
-            <frame_name>camera_link</frame_name>
-        </plugin>
-      </sensor>
-    </gazebo>
+  <!-- 카메라를 중간판(velodyne_mount_link) 위 11 cm 에 고정 -->
+  <joint name="camera_mount_joint" type="fixed">
+    <origin xyz="0.085 0 0.1415" rpy="0 0 0"/>
+    <parent link="velodyne_mount_link"/>
+    <child  link="camera_link"/>
+  </joint>
+  <!-- 카메라 링크(파란색 박스) -->
+  <link name="camera_link">
+    <inertial>
+      <origin xyz="0 0 0"/>
+      <mass value="0.1"/>
+      <inertia ixx="0.001" ixy="0" ixz="0" iyy="0.001" iyz="0" izz="0.001"/>
+    </inertial>
+    <visual>
+      <geometry>
+        <box size="0.02 0.1 0.007"/>
+      </geometry>
+      <material name="blue">
+        <color rgba="0 0 0.8 1"/>
+      </material>
+    </visual>
+    <collision>
+      <geometry>
+        <box size="0.05 0.05 0.05"/>
+      </geometry>
+    </collision>
+  </link>
+  <!-- Gazebo 센서 및 재질 정의 -->
+  <gazebo reference="camera_link">
+    <material>Gazebo/Blue</material>
+    <sensor name="color_camera" type="camera">
+      <camera>
+        <horizontal_fov>1.3962634</horizontal_fov>
+        <image>
+          <width>640</width>
+          <height>480</height>
+          <format>R8G8B8</format>
+        </image>
+        <clip><near>0.1</near><far>10</far></clip>
+      </camera>
+      <always_on>true</always_on>
+      <update_rate>30</update_rate>
+      <visualize>true</visualize>
+      <plugin name="color_camera_controller" filename="libgazebo_ros_camera.so">
+        <camera_name>camera</camera_name>
+        <image_topic_name>image_raw</image_topic_name>
+        <camera_info_topic_name>camera_info</camera_info_topic_name>
+        <frame_name>camera_link</frame_name>
+      </plugin>
+    </sensor>
+  </gazebo>
 </robot>

File: src/ugv_sim/scout_description/urdf/depth_camera.xacro (robot description, xacro)
@@ -1,60 +1,74 @@
 <?xml version="1.0"?>
-<robot xmlns:xacro="http://www.ros.org/wiki/xacro">
-    <!-- Depth 카메라 링크 추가 -->
-    <joint name="depth_camera_mount_joint" type="fixed">
-        <origin rpy="0 0 0" xyz="0 0 0.01"/>
-        <parent link="camera_link"/>
-        <child link="depth_camera_link"/>
-    </joint>
-    <link name="depth_camera_link">
-        <inertial>
-            <mass value="0.1"/>
-            <origin xyz="0 0 0"/>
-            <inertia ixx="0.001" ixy="0" ixz="0" iyy="0.001" iyz="0" izz="0.001"/>
-        </inertial>
-        <visual>
-            <geometry>
-                <box size="0.02 0.04 0.01"/>
-            </geometry>
-            <material name="white">
-                <color rgba="0.1 0.1 0.8 1.0"/>
-            </material>
-        </visual>
-        <collision>
-            <geometry>
-                <box size="0.05 0.05 0.05"/>
-            </geometry>
-        </collision>
-    </link>
-    <!-- Gazebo Depth 카메라 센서 -->
-    <gazebo reference="depth_camera_link">
-        <sensor name="depth_camera" type="depth">
-            <camera>
-                <horizontal_fov>1.3962634</horizontal_fov>
-                <image>
-                    <width>640</width>
-                    <height>480</height>
-                    <format>R8G8B8</format>
-                </image>
-                <depth_camera>
-                    <output>depth</output>
-                </depth_camera>
-                <clip>
-                    <near>0.1</near>
-                    <far>10</far>
-                </clip>
-            </camera>
-            <always_on>true</always_on>
-            <update_rate>30</update_rate>
-            <visualize>true</visualize>
-            <plugin name="depth_camera_controller" filename="libgazebo_ros_camera.so">
-                <camera_name>depth_camera</camera_name>
-                <image_topic_name>image_raw</image_topic_name>
-                <camera_info_topic_name>camera_info</camera_info_topic_name>
-                <depth_image_topic_name>depth/image_raw</depth_image_topic_name>
-                <depth_image_info_topic_name>depth/camera_info</depth_image_info_topic_name>
-                <frame_name>depth_camera_link</frame_name>
-            </plugin>
-        </sensor>
-    </gazebo>
+<robot xmlns:xacro="http://www.ros.org/wiki/xacro" name="depth_camera">
+  <link name="depth_camera_link">
+    <visual>
+      <origin xyz="0 0 0" rpy="0 0 0"/>
+      <geometry>
+        <box size="0.02 0.1 0.015"/>
+      </geometry>
+    </visual>
+    <collision>
+      <origin xyz="0 0 0" rpy="0 0 0"/>
+      <geometry>
+        <box size="0.05 0.05 0.05"/>
+      </geometry>
+    </collision>
+    <inertial>
+      <mass value="0.1"/>
+      <inertia ixx="0.0001" ixy="0.0" ixz="0.0" iyy="0.0001" iyz="0.0" izz="0.0001"/>
+    </inertial>
+  </link>
+  <joint name="depth_camera_joint" type="fixed">
+    <parent link="velodyne_mount_link"/>
+    <child link="depth_camera_link"/>
+    <origin xyz="0.085 0 0.1415" rpy="0 0 0"/>
+  </joint>
+  <link name="depth_camera_optical_link"/>
+  <joint name="depth_camera_optical_joint" type="fixed">
+    <parent link="depth_camera_link"/>
+    <child link="depth_camera_optical_link"/>
+    <origin xyz="0 0 0" rpy="${-pi/2} 0 ${-pi/2}"/>
+  </joint>
+  <gazebo reference="depth_camera_link">
+    <sensor type="depth" name="depth_camera">
+      <always_on>true</always_on>
+      <update_rate>30.0</update_rate>
+      <visualize>true</visualize>
+      <camera name="depth">
+        <horizontal_fov>1.047</horizontal_fov>
+        <image>
+          <width>640</width>
+          <height>480</height>
+          <format>R8G8B8</format>
+        </image>
+        <clip>
+          <near>0.1</near>
+          <far>10.0</far>
+        </clip>
+        <noise>
+          <type>gaussian</type>
+          <mean>0.0</mean>
+          <stddev>0.007</stddev>
+        </noise>
+      </camera>
+      <plugin name="depth_camera_controller" filename="libgazebo_ros_camera.so">
+        <alwaysOn>true</alwaysOn>
+        <updateRate>30.0</updateRate>
+        <cameraName>depth_camera</cameraName>
+        <frameName>depth_camera_optical_link</frameName>
+        <imageTopicName>depth/image_raw</imageTopicName>
+        <depthImageTopicName>depth/image_raw</depthImageTopicName>
+        <pointCloudTopicName>depth/points</pointCloudTopicName>
+        <cameraInfoTopicName>depth/camera_info</cameraInfoTopicName>
+        <depthImageCameraInfoTopicName>depth/camera_info</depthImageCameraInfoTopicName>
+        <pointCloudCutoff>0.1</pointCloudCutoff>
+        <pointCloudCutoffMax>10.0</pointCloudCutoffMax>
+        <distortionK1>0.0</distortionK1>
+        <distortionK2>0.0</distortionK2>
+        <distortionK3>0.0</distortionK3>
+        <distortionT1>0.0</distortionT1>
+        <distortionT2>0.0</distortionT2>
+      </plugin>
+    </sensor>
+  </gazebo>
 </robot>

File: src/ugv_sim/scout_description/urdf/mini.xacro (robot description, xacro)
@@ -9,8 +9,9 @@
     <xacro:include filename="$(find scout_description)/urdf/scout_mini_wheel_4.xacro" />
     <xacro:include filename="$(find scout_description)/urdf/mount.xacro" />
-    <!-- <xacro:include filename="$(find scout_description)/urdf/velodyne.xacro"/>       3D 라이다를 위한 Velodyne.xacro 추가 -->
-    <!-- <xacro:include filename="$(find scout_description)/urdf/laser.xacro"/>          2D 스캔을 위한 laser.xacro 추가 -->
-    <!-- <xacro:include filename="$(find scout_description)/urdf/camera.xacro"/>         camera.xacro 추가 -->
-    <!-- <xacro:include filename="$(find scout_description)/urdf/depth_camera.xacro"/>   depth_camera 추가 -->
+    <xacro:include filename="$(find scout_description)/urdf/velodyne.xacro"/>       <!-- 3D 라이다를 위한 Velodyne.xacro 추가 -->
+    <xacro:include filename="$(find scout_description)/urdf/laser.xacro"/>          <!-- 2D 스캔을 위한 laser.xacro 추가 -->
+    <xacro:include filename="$(find scout_description)/urdf/camera.xacro"/>         <!-- camera.xacro 추가 -->
+    <xacro:include filename="$(find scout_description)/urdf/depth_camera.xacro"/>   <!-- depth_camera 추가 -->
+    <!-- <xacro:include filename="$(find scout_description)/urdf/double_camera.xacro"/>   camera + depth camera 추가 -->
     <!-- Variables -->
     <xacro:property name="M_PI" value="3.14159"/>

File: src/ugv_sim/scout_description/urdf/mount.xacro (robot description, xacro)
@@ -12,9 +12,9 @@
   <xacro:property name="len_y_top" value="0.08"/>
   <!-- 실제 보이는 윗판(box) 크기 & 두께 -->
-  <xacro:property name="plate_x"  value="0.10"/>
-  <xacro:property name="plate_y"  value="0.10"/>
+  <xacro:property name="plate_x"  value="0.15"/>
+  <xacro:property name="plate_y"  value="0.15"/>
   <xacro:property name="th_top"   value="0.015"/>
   <!-- 기타 치수 -->
-  <xacro:property name="height"  value="0.12"/>
+  <xacro:property name="height"  value="0.13"/>
   <xacro:property name="beam_r"  value="0.004"/>
   <!-- 전체 오프셋 -->

File: src/ugv_sim/scout_description/urdf/velodyne.xacro (robot description, xacro)
@@ -2,5 +2,5 @@
 <robot xmlns:xacro="http://www.ros.org/wiki/xacro">
     <joint name="velodyne_base_mount_joint" type="fixed">
-        <origin rpy="0 0 0" xyz="0 0 0.055"/> <!-- 위치 조정 -->
+        <origin rpy="0 0 0" xyz="0 0 0.135"/> <!-- 위치 조정 -->
         <parent link="velodyne_mount_link"/>
         <child link="velodyne_base_link"/>

Commit message: simple_fix

File: src/ugv_sim/scout_description/urdf/camera.xacro (robot description, xacro)
@@ -18,6 +18,6 @@
         <box size="0.02 0.1 0.007"/>
       </geometry>
-      <material name="blue">
-        <color rgba="0 0 0.8 1"/>
+      <material name="red">
+        <color rgba="1 0 0 1"/>
       </material>
     </visual>
@@ -30,5 +30,5 @@
   <!-- Gazebo 센서 및 재질 정의 -->
   <gazebo reference="camera_link">
-    <material>Gazebo/Blue</material>
+    <material>Gazebo/Red</material>
     <sensor name="color_camera" type="camera">
       <camera>

File: src/ugv_sim/scout_description/urdf/depth_camera.xacro (robot description, xacro)
@@ -1,15 +1,25 @@
 <?xml version="1.0"?>
 <robot xmlns:xacro="http://www.ros.org/wiki/xacro" name="depth_camera">
+  <!-- 깊이 카메라를 로봇의 base_link에 고정 -->
+  <joint name="depth_camera_joint" type="fixed">
+    <origin xyz="0.085 0 0.135" rpy="0 0 0"/> <!-- 카메라 위치 (로봇 전방 10cm, 높이 10cm) -->
+    <parent link="velodyne_mount_link"/> <!-- 부모 링크 (로봇의 기준 링크로 변경 가능) -->
+    <child link="depth_camera_link"/>
+  </joint>
+  <!-- 깊이 카메라 링크 정의 -->
   <link name="depth_camera_link">
     <visual>
       <origin xyz="0 0 0" rpy="0 0 0"/>
       <geometry>
-        <box size="0.02 0.1 0.015"/>
+        <box size="0.02 0.1 0.007"/> <!-- 카메라의 시각적 표현 (임의의 박스) -->
       </geometry>
+      <material name="blue">
+        <color rgba="0 0 0.8 1"/>
+      </material>
     </visual>
     <collision>
       <origin xyz="0 0 0" rpy="0 0 0"/>
       <geometry>
-        <box size="0.05 0.05 0.05"/>
+        <box size="0.05 0.05 0.05"/> <!-- 충돌 모델 -->
       </geometry>
     </collision>
@@ -19,35 +29,26 @@
     </inertial>
   </link>
-  <joint name="depth_camera_joint" type="fixed">
-    <parent link="velodyne_mount_link"/>
-    <child link="depth_camera_link"/>
-    <origin xyz="0.085 0 0.1415" rpy="0 0 0"/>
-  </joint>
-  <link name="depth_camera_optical_link"/>
-  <joint name="depth_camera_optical_joint" type="fixed">
-    <parent link="depth_camera_link"/>
-    <child link="depth_camera_optical_link"/>
-    <origin xyz="0 0 0" rpy="${-pi/2} 0 ${-pi/2}"/>
-  </joint>
+  <!-- Gazebo 깊이 카메라 센서 정의 -->
   <gazebo reference="depth_camera_link">
+    <material>Gazebo/Blue</material>
     <sensor type="depth" name="depth_camera">
       <always_on>true</always_on>
-      <update_rate>30.0</update_rate>
-      <visualize>true</visualize>
+      <update_rate>30.0</update_rate> <!-- 초당 30Hz 업데이트 -->
+      <visualize>true</visualize> <!-- Gazebo에서 시각화 활성화 -->
       <camera name="depth">
-        <horizontal_fov>1.047</horizontal_fov>
+        <horizontal_fov>1.047</horizontal_fov> <!-- 약 60도 FOV -->
         <image>
           <width>640</width>
           <height>480</height>
-          <format>R8G8B8</format>
+          <format>R8G8B8</format> <!-- RGB 포맷 -->
         </image>
         <clip>
-          <near>0.1</near>
-          <far>10.0</far>
+          <near>0.1</near> <!-- 최소 거리 10cm -->
+          <far>10.0</far> <!-- 최대 거리 10m -->
         </clip>
         <noise>
           <type>gaussian</type>
           <mean>0.0</mean>
-          <stddev>0.007</stddev>
+          <stddev>0.007</stddev> <!-- 깊이 데이터에 가우시안 노이즈 추가 -->
         </noise>
       </camera>
@@ -56,5 +57,5 @@
         <updateRate>30.0</updateRate>
         <cameraName>depth_camera</cameraName>
-        <frameName>depth_camera_optical_link</frameName>
+        <frameName>depth_camera_link</frameName>
         <imageTopicName>depth/image_raw</imageTopicName>
         <depthImageTopicName>depth/image_raw</depthImageTopicName>
@@ -62,6 +63,6 @@
         <cameraInfoTopicName>depth/camera_info</cameraInfoTopicName>
         <depthImageCameraInfoTopicName>depth/camera_info</depthImageCameraInfoTopicName>
-        <pointCloudCutoff>0.1</pointCloudCutoff>
-        <pointCloudCutoffMax>10.0</pointCloudCutoffMax>
+        <pointCloudCutoff>0.1</pointCloudCutoff> <!-- 포인트 클라우드 최소 거리 -->
+        <pointCloudCutoffMax>10.0</pointCloudCutoffMax> <!-- 포인트 클라우드 최대 거리 -->
         <distortionK1>0.0</distortionK1>
         <distortionK2>0.0</distortionK2>

Commit message: simple_fix

File: src/ugv_sim/scout_description/urdf/camera.xacro (robot description, xacro)
@@ -1,7 +1,6 @@
 <?xml version="1.0"?>
 <robot xmlns:xacro="http://www.ros.org/wiki/xacro">
-  <!-- 카메라를 중간판(velodyne_mount_link) 위 11 cm 에 고정 -->
   <joint name="camera_mount_joint" type="fixed">
-    <origin xyz="0.085 0 0.1415" rpy="0 0 0"/>
+    <origin xyz="0.085 0 0.232" rpy="0 0 0"/>
     <parent link="velodyne_mount_link"/>
     <child  link="camera_link"/>

File: src/ugv_sim/scout_description/urdf/depth_camera.xacro (robot description, xacro)
@@ -1,7 +1,6 @@
 <?xml version="1.0"?>
 <robot xmlns:xacro="http://www.ros.org/wiki/xacro" name="depth_camera">
-  <!-- 깊이 카메라를 로봇의 base_link에 고정 -->
   <joint name="depth_camera_joint" type="fixed">
-    <origin xyz="0.085 0 0.135" rpy="0 0 0"/> <!-- 카메라 위치 (로봇 전방 10cm, 높이 10cm) -->
+    <origin xyz="0.085 0 0.239" rpy="0 0 0"/>
     <parent link="velodyne_mount_link"/> <!-- 부모 링크 (로봇의 기준 링크로 변경 가능) -->
     <child link="depth_camera_link"/>

File: src/ugv_sim/scout_description/urdf/mount.xacro (robot description, xacro)
@@ -16,5 +16,5 @@
   <xacro:property name="th_top"   value="0.015"/>
   <!-- 기타 치수 -->
-  <xacro:property name="height"  value="0.13"/>
+  <xacro:property name="height"  value="0.228"/>
   <xacro:property name="beam_r"  value="0.004"/>
   <!-- 전체 오프셋 -->

File: src/ugv_sim/scout_description/urdf/velodyne.xacro (robot description, xacro)
@@ -2,5 +2,5 @@
 <robot xmlns:xacro="http://www.ros.org/wiki/xacro">
     <joint name="velodyne_base_mount_joint" type="fixed">
-        <origin rpy="0 0 0" xyz="0 0 0.135"/> <!-- 위치 조정 -->
+        <origin rpy="0 0 0" xyz="0 0 0.243"/> <!-- 위치 조정 -->
         <parent link="velodyne_mount_link"/>
         <child link="velodyne_base_link"/>
