Commit message: simple_fix

File: src/ugv_sim/scout_description/urdf/gripper.xacro (robot description, xacro)
@@ -1,5 +1,5 @@
 <?xml version="1.0"?>
 <robot name="scout_mini_gripper" xmlns:xacro="http://ros.org/wiki/xacro">
-  <xacro:macro name="scout_mini_gripper" params="parent mount_x:=0.40 mount_y:=0.0 mount_z:=0.20 opening_max:=0.18">
+  <xacro:macro name="scout_mini_gripper" params="parent mount_x:=0.15 mount_y:=0.0 mount_z:=0.1 opening_max:=0.18">
     <xacro:property name="finger_len" value="0.20"/>
     <xacro:property name="finger_thk" value="0.02"/>
@@ -9,12 +9,12 @@
     <xacro:property name="open_default" value="0.06"/>
     <xacro:property name="brace_thk" value="0.02"/>
-    <xacro:property name="pillar_len" value="${mount_z}"/>   <!-- 세로(높이) -->
-    <xacro:property name="arm_len"    value="${mount_x}"/>   <!-- 가로(전방) -->
-    <link name="gripper_pillar">
+    <xacro:property name="connecter_h" value="${mount_z}"/>   <!-- 세로(높이) -->
+    <xacro:property name="connecter_l"    value="${mount_x}"/>   <!-- 가로(전방) -->
+    <link name="gripper_connecter">
       <visual>
-        <geometry><box size="${brace_thk} ${brace_thk} ${pillar_len}"/></geometry>
+        <geometry><box size="${brace_thk} ${brace_thk} ${connecter_h}"/></geometry>
         <material name="Grey"><color rgba="0.5 0.5 0.5 1.0"/></material>
       </visual>
-      <collision><geometry><box size="${brace_thk} ${brace_thk} ${pillar_len}"/></geometry></collision>
+      <collision><geometry><box size="${brace_thk} ${brace_thk} ${connecter_h}"/></geometry></collision>
       <inertial>
         <mass value="0.2"/>
@@ -23,15 +23,15 @@
       </inertial>
     </link>
-    <joint name="gripper_pillar_mount" type="fixed">
+    <joint name="gripper_connecter_mount" type="fixed">
       <parent link="${parent}"/>
-      <child  link="gripper_pillar"/>
-      <origin xyz="0 ${mount_y} ${pillar_len/2.0}" rpy="0 0 0"/>
+      <child  link="gripper_connecter"/>
+      <origin xyz="0.18 ${mount_y} ${connecter_h/2.0}" rpy="0 0 0"/>
     </joint>
     <link name="gripper_arm">
       <visual>
-        <geometry><box size="${arm_len} ${brace_thk} ${brace_thk}"/></geometry>
+        <geometry><box size="${connecter_l} ${brace_thk} ${brace_thk}"/></geometry>
         <material name="Grey"><color rgba="0.5 0.5 0.5 1.0"/></material>
       </visual>
-      <collision><geometry><box size="${arm_len} ${brace_thk} ${brace_thk}"/></geometry></collision>
+      <collision><geometry><box size="${connecter_l} ${brace_thk} ${brace_thk}"/></geometry></collision>
       <inertial>
         <mass value="0.15"/>
@@ -40,8 +40,8 @@
       </inertial>
     </link>
-    <joint name="pillar_to_arm" type="fixed">
-      <parent link="gripper_pillar"/>
+    <joint name="connecter_to_arm" type="fixed">
+      <parent link="gripper_connecter"/>
       <child  link="gripper_arm"/>
-      <origin xyz="${arm_len/2.0} 0 ${pillar_len/2.0}" rpy="0 0 0"/>
+      <origin xyz="${connecter_l/2.0} 0 ${connecter_h/2.0}" rpy="0 0 0"/>
     </joint>
     <link name="gripper_base">
@@ -60,5 +60,5 @@
       <parent link="gripper_arm"/>
       <child  link="gripper_base"/>
-      <origin xyz="${arm_len/2.0} 0 0" rpy="0 0 0"/>
+      <origin xyz="${connecter_l/2.0} 0 0" rpy="0 0 0"/>
     </joint>
     <link name="left_finger">
@@ -120,4 +120,10 @@
     </ros2_control>
   </xacro:macro>
+  <gazebo reference="connecter_to_arm">
+    <material>Gazebo/Grey</material>
+  </gazebo>
+    <gazebo reference="gripper_connecter_mount">
+  <material>Gazebo/Grey</material>
+  </gazebo>
   <gazebo reference="gripper_base">
     <material>Gazebo/Grey</material>

File: src/ugv_sim/scout_description/urdf/mini.xacro (robot description, xacro)
@@ -113,5 +113,5 @@
     <!-- Gazebo definitions  -->
     <xacro:include filename="$(find scout_description)/urdf/scout_mini.gazebo" />
-    <xacro:scout_mini_gripper parent="base_link" mount_x="0.40" mount_y="0.0" mount_z="0.13" opening_max="0.18"/>
+    <xacro:scout_mini_gripper parent="base_link" mount_x="0.15" mount_y="0.0" mount_z="0.1" opening_max="0.20"/>
     <gazebo>
         <plugin name="gazebo_ros2_control" filename="libgazebo_ros2_control.so">

Commit message: connecter_up_and_down

File: src/ugv_sim/scout_description/urdf/gripper.xacro (robot description, xacro)
@@ -13,5 +13,5 @@
     <link name="gripper_connecter">
       <visual>
-        <geometry><box size="${brace_thk} ${brace_thk} ${connecter_h}"/></geometry>
+        <geometry><box size="${brace_thk} ${brace_thk} 0.2"/></geometry>
         <material name="Grey"><color rgba="0.5 0.5 0.5 1.0"/></material>
       </visual>
@@ -40,8 +40,11 @@
       </inertial>
     </link>
-    <joint name="connecter_to_arm" type="fixed">
+    <joint name="connecter_to_arm" type="prismatic">
       <parent link="gripper_connecter"/>
       <child  link="gripper_arm"/>
       <origin xyz="${connecter_l/2.0} 0 ${connecter_h/2.0}" rpy="0 0 0"/>
+      <axis xyz="0 0 1"/>
+      <limit lower="-0.05" upper="0.05" effort="200" velocity="0.5"/>
+      <dynamics damping="5.0" friction="0.1"/>
     </joint>
     <link name="gripper_base">
@@ -118,4 +121,10 @@
         <state_interface name="effort"/>
       </joint>
+      <joint name="connecter_to_arm">
+        <command_interface name="position"/>
+        <state_interface name="position"/>
+        <state_interface name="velocity"/>
+        <state_interface name="effort"/>
+      </joint>
     </ros2_control>
   </xacro:macro>

Commit message: update_gripper

File: src/ugv_sim/scout_description/urdf/gripper.xacro (robot description, xacro)
@@ -1,5 +1,5 @@
 <?xml version="1.0"?>
 <robot name="scout_mini_gripper" xmlns:xacro="http://ros.org/wiki/xacro">
-  <xacro:macro name="scout_mini_gripper" params="parent mount_x:=0.15 mount_y:=0.0 mount_z:=0.1 opening_max:=0.18">
+  <xacro:macro name="scout_mini_gripper" params="parent mount_x:=0.15 mount_y:=0.1 mount_z:=0.1 opening_max:=0.3">
     <xacro:property name="finger_len" value="0.20"/>
     <xacro:property name="finger_thk" value="0.02"/>
@@ -7,14 +7,22 @@
     <xacro:property name="half_thk" value="${finger_thk/2.0}"/>
     <xacro:property name="half_gap" value="${closed_gap/2.0}"/>
-    <xacro:property name="open_default" value="0.06"/>
+    <xacro:property name="open_default" value="0.09"/>
     <xacro:property name="brace_thk" value="0.02"/>
-    <xacro:property name="connecter_h" value="${mount_z}"/>   <!-- 세로(높이) -->
-    <xacro:property name="connecter_l"    value="${mount_x}"/>   <!-- 가로(전방) -->
+    <xacro:property name="connecter_h" value="${mount_z}"/>
+    <xacro:property name="connecter_l" value="${mount_x}"/>
     <link name="gripper_connecter">
       <visual>
-        <geometry><box size="${brace_thk} ${brace_thk} 0.2"/></geometry>
-        <material name="Grey"><color rgba="0.5 0.5 0.5 1.0"/></material>
-      </visual>
-      <collision><geometry><box size="${brace_thk} ${brace_thk} ${connecter_h}"/></geometry></collision>
+        <geometry>
+          <box size="${brace_thk} ${brace_thk} 0.12"/>
+        </geometry>
+        <material name="DarkGrey">
+          <color rgba="0.4 0.4 0.4 1.0"/>
+        </material>
+      </visual>
+      <collision>
+        <geometry>
+          <box size="${brace_thk} ${brace_thk} ${connecter_h + 0.02}"/>
+        </geometry>
+      </collision>
       <inertial>
         <mass value="0.2"/>
@@ -26,15 +34,23 @@
       <parent link="${parent}"/>
       <child  link="gripper_connecter"/>
-      <origin xyz="0.18 ${mount_y} ${connecter_h/2.0}" rpy="0 0 0"/>
+      <origin xyz="0.18 ${mount_y} ${connecter_h/2.0 + 0.03}" rpy="0 0 0"/>
     </joint>
     <link name="gripper_arm">
       <visual>
-        <geometry><box size="${connecter_l} ${brace_thk} ${brace_thk}"/></geometry>
-        <material name="Grey"><color rgba="0.5 0.5 0.5 1.0"/></material>
-      </visual>
-      <collision><geometry><box size="${connecter_l} ${brace_thk} ${brace_thk}"/></geometry></collision>
+        <geometry>
+          <box size="${connecter_l} ${brace_thk} ${brace_thk}"/>
+        </geometry>
+        <material name="DarkGrey">
+          <color rgba="0.4 0.4 0.4 1.0"/>
+        </material>
+      </visual>
+      <collision>
+        <geometry>
+          <box size="${connecter_l} ${brace_thk} ${brace_thk}"/>
+        </geometry>
+      </collision>
       <inertial>
         <mass value="0.15"/>
-        <origin xyz="0 0 0"/>
+        <origin xyz="-0 0 0"/>
         <inertia ixx="0.00005" iyy="0.00005" izz="0.00002" ixy="0" ixz="0" iyz="0"/>
       </inertial>
@@ -43,15 +59,46 @@
       <parent link="gripper_connecter"/>
       <child  link="gripper_arm"/>
-      <origin xyz="${connecter_l/2.0} 0 ${connecter_h/2.0}" rpy="0 0 0"/>
+      <origin xyz="${connecter_l/2.0} 0 ${connecter_h/2.0 - 0.03}" rpy="0 0 0"/>
       <axis xyz="0 0 1"/>
-      <limit lower="-0.05" upper="0.05" effort="200" velocity="0.5"/>
+      <limit lower="-0.04" upper="0.02" effort="200" velocity="0.4"/>
       <dynamics damping="5.0" friction="0.1"/>
     </joint>
+    <link name="arm_vertical">
+        <visual>
+            <geometry>
+                <box size="${brace_thk} ${brace_thk} 0.15"/>
+            </geometry>
+            <material name="DarkGrey">
+                <color rgba="0.4 0.4 0.4 1.0"/>
+            </material>
+        </visual>
+        <collision>
+            <geometry>
+                <box size="${brace_thk} ${brace_thk} 0.15"/>
+            </geometry>
+        </collision>
+        <inertial>
+            <mass value="0.1"/>
+            <origin xyz="0 0 0"/>
+            <inertia ixx="0.00002" iyy="0.00002" izz="0.00002" ixy="0" ixz="0" iyz="0"/>
+        </inertial>
+    </link>
+    <joint name="arm_to_vertical" type="fixed">
+        <parent link="gripper_arm"/>
+        <child link="arm_vertical"/>
+        <origin xyz="${connecter_l/2.0} 0 ${-0.15/2.0 - brace_thk/2.0 + 0.02}" rpy="0 0 0"/>
+    </joint>
     <link name="gripper_base">
       <visual>
-        <geometry><box size="0.02 0.25 0.05"/></geometry>
-        <material name="Grey"><color rgba="0.5 0.5 0.5 1.0"/></material>
-      </visual>
-      <collision><geometry><box size="0.02 0.25 0.05"/></geometry></collision>
+        <geometry><box size="0.02 0.3 0.05"/></geometry>
+        <material name="DarkGrey">
+          <color rgba="0.4 0.4 0.4 1.0"/>
+        </material>
+      </visual>
+      <collision>
+        <geometry>
+          <box size="0.02 0.33 0.05"/>
+        </geometry>
+      </collision>
       <inertial>
         <mass value="0.5"/>
@@ -60,15 +107,23 @@
       </inertial>
     </link>
-    <joint name="arm_to_gripper_base" type="fixed">
-      <parent link="gripper_arm"/>
+    <joint name="vertical_to_gripper_base" type="fixed">
+      <parent link="arm_vertical"/>
       <child  link="gripper_base"/>
-      <origin xyz="${connecter_l/2.0} 0 0" rpy="0 0 0"/>
+      <origin xyz="0 0 -0.075" rpy="0 0 0"/>
     </joint>
     <link name="left_finger">
       <visual>
-        <geometry><box size="${finger_len} ${finger_thk} 0.04"/></geometry>
-        <material name="Grey"><color rgba="0.5 0.5 0.5 1.0"/></material>
-      </visual>
-      <collision><geometry><box size="${finger_len} ${finger_thk} 0.04"/></geometry></collision>
+        <geometry>
+          <box size="${finger_len} ${finger_thk} 0.04"/>
+        </geometry>
+        <material name="DarkGrey">
+          <color rgba="0.4 0.4 0.4 1.0"/>
+        </material>
+      </visual>
+      <collision>
+        <geometry>
+          <box size="${finger_len} ${finger_thk} 0.04"/>
+        </geometry>
+      </collision>
       <inertial>
         <mass value="0.2"/>
@@ -85,10 +140,43 @@
       <dynamics damping="5.0" friction="0.1"/>
     </joint>
+    <link name="left_finger_stopper">
+      <visual>
+        <geometry>
+          <box size="0.02 0.04 0.04"/>
+        </geometry>
+        <material name="DarkGrey">
+          <color rgba="0.2 0.2 0.2 1.0"/>
+        </material>
+      </visual>
+      <collision>
+        <geometry>
+          <box size="0.01 0.015 0.04"/>
+        </geometry>
+      </collision>
+      <inertial>
+        <mass value="0.01"/>
+        <origin xyz="0 0 0"/>
+        <inertia ixx="0.000001" iyy="0.000001" izz="0.000001" ixy="0" ixz="0" iyz="0"/>
+      </inertial>
+    </link>
+    <joint name="left_finger_stopper_joint" type="fixed">
+      <parent link="left_finger"/>
+      <child  link="left_finger_stopper"/>
+      <origin xyz="0.1 -0.01 0"/>
+    </joint>
     <link name="right_finger">
       <visual>
-        <geometry><box size="${finger_len} ${finger_thk} 0.04"/></geometry>
-        <material name="Grey"><color rgba="0.5 0.5 0.5 1.0"/></material>
-      </visual>
-      <collision><geometry><box size="${finger_len} ${finger_thk} 0.04"/></geometry></collision>
+        <geometry>
+          <box size="${finger_len} ${finger_thk} 0.04"/>
+        </geometry>
+        <material name="DarkGrey">
+          <color rgba="0.4 0.4 0.4 1.0"/>
+        </material>
+      </visual>
+      <collision>
+        <geometry>
+          <box size="${finger_len} ${finger_thk} 0.04"/>
+        </geometry>
+      </collision>
       <inertial>
         <mass value="0.2"/>
@@ -104,4 +192,29 @@
       <limit lower="${-open_default}" upper="${opening_max/2.0 - open_default}" effort="200" velocity="1.0"/>
       <dynamics damping="5.0" friction="0.1"/>
+    </joint>
+    <link name="right_finger_stopper">
+      <visual>
+        <geometry>
+          <box size="0.02 0.04 0.04"/>
+        </geometry>
+        <material name="DarkGrey">
+          <color rgba="0.2 0.2 0.2 1.0"/>
+        </material>
+      </visual>
+      <collision>
+        <geometry>
+          <box size="0.01 0.015 0.04"/>
+        </geometry>
+      </collision>
+      <inertial>
+        <mass value="0.01"/>
+        <origin xyz="0 0 0"/>
+        <inertia ixx="0.000001" iyy="0.000001" izz="0.000001" ixy="0" ixz="0" iyz="0"/>
+      </inertial>
+    </link>
+    <joint name="right_finger_stopper_joint" type="fixed">
+      <parent link="right_finger"/>
+      <child  link="right_finger_stopper"/>
+      <origin xyz="0.1 0.01 0"/>
     </joint>
     <ros2_control name="gripper_ros2_control" type="system">
@@ -129,18 +242,27 @@
     </ros2_control>
   </xacro:macro>
-  <gazebo reference="connecter_to_arm">
-    <material>Gazebo/Grey</material>
-  </gazebo>
-    <gazebo reference="gripper_connecter_mount">
-  <material>Gazebo/Grey</material>
+  <gazebo reference="gripper_connecter">
+    <material>Gazebo/DarkGrey</material>
+  </gazebo>
+  <gazebo reference="gripper_arm">
+    <material>Gazebo/DarkGrey</material>
+  </gazebo>
+  <gazebo reference="arm_vertical">
+    <material>Gazebo/DarkGrey</material>
   </gazebo>
   <gazebo reference="gripper_base">
-    <material>Gazebo/Grey</material>
-  </gazebo>
-    <gazebo reference="left_finger">
-  <material>Gazebo/Grey</material>
+    <material>Gazebo/DarkGrey</material>
+  </gazebo>
+  <gazebo reference="left_finger">
+  <material>Gazebo/DarkGrey</material>
+  </gazebo>
+  <gazebo reference="left_finger_stopper">
+    <material>Gazebo/Black</material>
   </gazebo>
   <gazebo reference="right_finger">
-    <material>Gazebo/Grey</material>
+    <material>Gazebo/DarkGrey</material>
+  </gazebo>
+  <gazebo reference="right_finger_stopper">
+    <material>Gazebo/Black</material>
   </gazebo>
 </robot>

File: src/ugv_sim/scout_description/urdf/mini.xacro (robot description, xacro)
@@ -113,5 +113,5 @@
     <!-- Gazebo definitions  -->
     <xacro:include filename="$(find scout_description)/urdf/scout_mini.gazebo" />
-    <xacro:scout_mini_gripper parent="base_link" mount_x="0.15" mount_y="0.0" mount_z="0.1" opening_max="0.20"/>
+    <xacro:scout_mini_gripper parent="base_link" mount_x="0.15" mount_y="0.0" mount_z="0.12" opening_max="0.6"/>
     <gazebo>
         <plugin name="gazebo_ros2_control" filename="libgazebo_ros2_control.so">

Commit message: simple_fix

File: src/ugv_sim/scout_description/urdf/gripper.xacro (robot description, xacro)
@@ -151,5 +151,5 @@
       <collision>
         <geometry>
-          <box size="0.01 0.015 0.04"/>
+          <box size="0.02 0.04 0.04"/>
         </geometry>
       </collision>
@@ -204,5 +204,5 @@
       <collision>
         <geometry>
-          <box size="0.01 0.015 0.04"/>
+          <box size="0.02 0.04 0.04"/>
         </geometry>
       </collision>
