Commit message: update_2D_laser

File: src/ugv_sim/scout_description/urdf/mini.xacro (robot description, xacro)
@@ -8,4 +8,6 @@
     <xacro:include filename="$(find scout_description)/urdf/scout_mini_wheel_3.xacro" />
     <xacro:include filename="$(find scout_description)/urdf/scout_mini_wheel_4.xacro" />
+    <xacro:include filename="$(find scout_description)/urdf/velodyne.xacro"/>
+    <xacro:include filename="$(find scout_description)/urdf/laser.xacro"/>
     <!-- Variables -->
     <xacro:property name="M_PI" value="3.14159"/>

File: src/ugv_sim/scout_description/urdf/velodyne.xacro (robot description, xacro)
@@ -2,5 +2,5 @@
 <robot xmlns:xacro="http://www.ros.org/wiki/xacro">
     <joint name="velodyne_base_mount_joint" type="fixed">
-        <origin rpy="0 0 0" xyz="0 0 0.06"/> <!-- 위치 조정 -->
+        <origin rpy="0 0 0" xyz="0 0 0.055"/> <!-- 위치 조정 -->
         <parent link="base_link"/>
         <child link="velodyne_base_link"/>

Commit message: update_costmap

File: src/ugv_sim/scout_description/urdf/mini.xacro (robot description, xacro)
@@ -8,8 +8,8 @@
     <xacro:include filename="$(find scout_description)/urdf/scout_mini_wheel_3.xacro" />
     <xacro:include filename="$(find scout_description)/urdf/scout_mini_wheel_4.xacro" />
-    <xacro:include filename="$(find scout_description)/urdf/velodyne.xacro"/>
-    <xacro:include filename="$(find scout_description)/urdf/laser.xacro"/>
-    <xacro:include filename="$(find scout_description)/urdf/camera.xacro"/>
-    <xacro:include filename="$(find scout_description)/urdf/depth_camera.xacro"/>
+    <xacro:include filename="$(find scout_description)/urdf/velodyne.xacro"/>       <!-- 3D 라이다를 위한 Velodyne.xacro 추가 -->
+    <xacro:include filename="$(find scout_description)/urdf/laser.xacro"/>          <!-- 2D 스캔을 위한 laser.xacro 추가 -->
+    <xacro:include filename="$(find scout_description)/urdf/camera.xacro"/>         <!-- camera.xacro 추가 -->
+    <xacro:include filename="$(find scout_description)/urdf/depth_camera.xacro"/>   <!-- depth_camera 추가 -->
     <!-- Variables -->
     <xacro:property name="M_PI" value="3.14159"/>
@@ -97,4 +97,11 @@
         <origin xyz="${-wheelbase/2} ${-track/2} ${wheel_vertical_offset+0.001}" rpy="1.57 0 0" />
     </xacro:scout_mini_wheel_4>
+    <!--  base_footprint frame  -->
+    <link name="base_footprint"/>
+        <joint name="base_footprint_joint" type="fixed">
+        <parent link="base_link"/>
+        <child  link="base_footprint"/>
+        <origin xyz="0 0 0" rpy="0 0 0"/>
+    </joint>
     <!-- Additional definitions -->
     <xacro:include filename="$(arg urdf_extras)" />

Commit message: create_mount.xacro

File: src/ugv_sim/scout_description/urdf/mini.xacro (robot description, xacro)
@@ -8,8 +8,9 @@
     <xacro:include filename="$(find scout_description)/urdf/scout_mini_wheel_3.xacro" />
     <xacro:include filename="$(find scout_description)/urdf/scout_mini_wheel_4.xacro" />
-    <xacro:include filename="$(find scout_description)/urdf/velodyne.xacro"/>       <!-- 3D 라이다를 위한 Velodyne.xacro 추가 -->
-    <xacro:include filename="$(find scout_description)/urdf/laser.xacro"/>          <!-- 2D 스캔을 위한 laser.xacro 추가 -->
-    <xacro:include filename="$(find scout_description)/urdf/camera.xacro"/>         <!-- camera.xacro 추가 -->
-    <xacro:include filename="$(find scout_description)/urdf/depth_camera.xacro"/>   <!-- depth_camera 추가 -->
+    <xacro:include filename="$(find scout_description)/urdf/mount.xacro" />
+    <!-- <xacro:include filename="$(find scout_description)/urdf/velodyne.xacro"/>       3D 라이다를 위한 Velodyne.xacro 추가 -->
+    <!-- <xacro:include filename="$(find scout_description)/urdf/laser.xacro"/>          2D 스캔을 위한 laser.xacro 추가 -->
+    <!-- <xacro:include filename="$(find scout_description)/urdf/camera.xacro"/>         camera.xacro 추가 -->
+    <!-- <xacro:include filename="$(find scout_description)/urdf/depth_camera.xacro"/>   depth_camera 추가 -->
     <!-- Variables -->
     <xacro:property name="M_PI" value="3.14159"/>
@@ -98,4 +99,6 @@
     </xacro:scout_mini_wheel_4>
     <!--  base_footprint frame  -->
+    <!-- front_laser -> base_footprint 변환 관련 TF 오류 수정용 -->
+    <!-- Couldn't transform from front_laser to base_footprint … -->
     <link name="base_footprint"/>
         <joint name="base_footprint_joint" type="fixed">

File: src/ugv_sim/scout_description/urdf/velodyne.xacro (robot description, xacro)
@@ -3,5 +3,5 @@
     <joint name="velodyne_base_mount_joint" type="fixed">
         <origin rpy="0 0 0" xyz="0 0 0.055"/> <!-- 위치 조정 -->
-        <parent link="base_link"/>
+        <parent link="velodyne_mount_link"/>
         <child link="velodyne_base_link"/>
     </joint>

Commit message: fix_base_link_to_mount

File: src/ugv_sim/scout_description/urdf/mini.xacro (robot description, xacro)
@@ -23,5 +23,5 @@
     <xacro:property name="wheelbase" value="0.463951"/>
     <xacro:property name="track" value="0.416503"/>
-    <xacro:property name="wheel_vertical_offset" value="-0.100998" />
+    <xacro:property name="wheel_vertical_offset" value="-0.077" />
 <!--    <xacro:property name="track" value="0.3426" />
     <xacro:property name="wheelbase" value="0.3181"/>
