Commit message: error_fix

File: src/ugv_sim/scout_description/urdf/depth_camera.xacro (robot description, xacro)
@@ -11,7 +11,5 @@
             <mass value="0.1"/>
             <origin xyz="0 0 0"/>
-            <inertia ixx="0.001" ixy="0" ixz="0"
-                     iyy="0.001" iyz="0"
-                     izz="0.001"/>
+            <inertia ixx="0.001" ixy="0" ixz="0" iyy="0.001" iyz="0" izz="0.001"/>
         </inertial>
         <visual>
@@ -19,9 +17,6 @@
                 <box size="0.02 0.04 0.01"/>
             </geometry>
-            <material name="depth_camera_gray">
-                <ambient>0.5 0.5 0.5 1</ambient>
-                <diffuse>0.5 0.5 0.5 1</diffuse>
-                <specular>0.1 0.1 0.1 1</specular>
-                <emissive>0 0 0 1</emissive>
+            <material name="white">
+                <color rgba="0.1 0.1 0.8 1.0"/>
             </material>
         </visual>

File: src/ugv_sim/scout_description/urdf/mini.xacro (robot description, xacro)
@@ -10,4 +10,6 @@
     <xacro:include filename="$(find scout_description)/urdf/velodyne.xacro"/>
     <xacro:include filename="$(find scout_description)/urdf/laser.xacro"/>
+    <xacro:include filename="$(find scout_description)/urdf/camera.xacro"/>
+    <xacro:include filename="$(find scout_description)/urdf/depth_camera.xacro"/>
     <!-- Variables -->
     <xacro:property name="M_PI" value="3.14159"/>

File: src/ugv_sim/scout_description/urdf/scout_mini.xacro (robot description, xacro)
@@ -7,5 +7,5 @@
     <xacro:include filename="$(find scout_description)/urdf/scout_mini_wheel_2.xacro" />
     <xacro:include filename="$(find scout_description)/urdf/scout_mini_wheel_3.xacro" />
-    <xacro:include filename="$(find scout_description)/urdf/scout_mini_wheel_4.xacro" />
+    <xacro:include filename="$(find scout_description)/urdf/scout_mini_wheel_4.xacro" />zz
     <!-- Variables -->
     <xacro:property name="M_PI" value="3.14159"/>

Commit message: simple_fix

File: src/ugv_sim/scout_description/urdf/depth_camera.xacro (robot description, xacro)
@@ -3,23 +3,16 @@
   <joint name="depth_camera_joint" type="fixed">
     <origin xyz="0.085 0 0.239" rpy="0 0 0"/>
-    <parent link="velodyne_mount_link"/> <!-- 부모 링크 (로봇의 기준 링크로 변경 가능) -->
+    <parent link="velodyne_mount_link"/>
     <child link="depth_camera_link"/>
   </joint>
-  <!-- 깊이 카메라 링크 정의 -->
   <link name="depth_camera_link">
     <visual>
       <origin xyz="0 0 0" rpy="0 0 0"/>
-      <geometry>
-        <box size="0.02 0.1 0.007"/> <!-- 카메라의 시각적 표현 (임의의 박스) -->
-      </geometry>
-      <material name="blue">
-        <color rgba="0 0 0.8 1"/>
-      </material>
+      <geometry><box size="0.02 0.10 0.007"/></geometry>
+      <material name="blue"><color rgba="0 0 0.8 1"/></material>
     </visual>
     <collision>
       <origin xyz="0 0 0" rpy="0 0 0"/>
-      <geometry>
-        <box size="0.05 0.05 0.05"/> <!-- 충돌 모델 -->
-      </geometry>
+      <geometry><box size="0.05 0.05 0.05"/></geometry>
     </collision>
     <inertial>
@@ -28,26 +21,50 @@
     </inertial>
   </link>
-  <!-- Gazebo 깊이 카메라 센서 정의 -->
+  <link name="depth_camera_optical_frame"/>
+  <joint name="depth_camera_optical_joint" type="fixed">
+    <parent link="depth_camera_link"/>
+    <child link="depth_camera_optical_frame"/>
+    <origin xyz="0 0 0" rpy="-1.57079632679 0 -1.57079632679"/>
+  </joint>
   <gazebo reference="depth_camera_link">
     <material>Gazebo/Blue</material>
-    <sensor type="depth" name="depth_camera">
+    <sensor type="camera" name="depth_camera_rgb">
       <always_on>true</always_on>
-      <update_rate>30.0</update_rate> <!-- 초당 30Hz 업데이트 -->
-      <visualize>true</visualize> <!-- Gazebo에서 시각화 활성화 -->
-      <camera name="depth">
-        <horizontal_fov>1.047</horizontal_fov> <!-- 약 60도 FOV -->
+      <update_rate>30.0</update_rate>
+      <visualize>true</visualize>
+      <camera name="rgb">
+        <horizontal_fov>1.047</horizontal_fov>
         <image>
           <width>640</width>
           <height>480</height>
-          <format>R8G8B8</format> <!-- RGB 포맷 -->
+          <format>R8G8B8</format>
         </image>
-        <clip>
-          <near>0.1</near> <!-- 최소 거리 10cm -->
-          <far>10.0</far> <!-- 최대 거리 10m -->
-        </clip>
+        <clip><near>0.1</near><far>10.0</far></clip>
+      </camera>
+      <plugin name="rgb_camera_controller" filename="libgazebo_ros_camera.so">
+        <alwaysOn>true</alwaysOn>
+        <updateRate>30.0</updateRate>
+        <cameraName>depth_camera</cameraName>
+        <frameName>depth_camera_optical_frame</frameName>
+        <imageTopicName>image_raw</imageTopicName>
+        <cameraInfoTopicName>camera_info</cameraInfoTopicName>
+      </plugin>
+    </sensor>
+    <sensor type="depth" name="depth_camera_depth">
+      <always_on>true</always_on>
+      <update_rate>30.0</update_rate>
+      <visualize>true</visualize>
+      <camera name="depth">
+        <horizontal_fov>1.047</horizontal_fov>
+        <image>
+          <width>640</width>
+          <height>480</height>
+          <format>R8G8B8</format>
+        </image>
+        <clip><near>0.1</near><far>10.0</far></clip>
         <noise>
           <type>gaussian</type>
           <mean>0.0</mean>
-          <stddev>0.007</stddev> <!-- 깊이 데이터에 가우시안 노이즈 추가 -->
+          <stddev>0.007</stddev>
         </noise>
       </camera>
@@ -56,12 +73,10 @@
         <updateRate>30.0</updateRate>
         <cameraName>depth_camera</cameraName>
-        <frameName>depth_camera_link</frameName>
-        <imageTopicName>depth/image_raw</imageTopicName>
+        <frameName>depth_camera_optical_frame</frameName>
         <depthImageTopicName>depth/image_raw</depthImageTopicName>
-        <pointCloudTopicName>depth/points</pointCloudTopicName>
-        <cameraInfoTopicName>depth/camera_info</cameraInfoTopicName>
         <depthImageCameraInfoTopicName>depth/camera_info</depthImageCameraInfoTopicName>
-        <pointCloudCutoff>0.1</pointCloudCutoff> <!-- 포인트 클라우드 최소 거리 -->
-        <pointCloudCutoffMax>10.0</pointCloudCutoffMax> <!-- 포인트 클라우드 최대 거리 -->
+        <pointCloudTopicName>points</pointCloudTopicName>
+        <pointCloudCutoff>0.1</pointCloudCutoff>
+        <pointCloudCutoffMax>10.0</pointCloudCutoffMax>
         <distortionK1>0.0</distortionK1>
         <distortionK2>0.0</distortionK2>

File: src/ugv_sim/scout_description/urdf/mini.xacro (robot description, xacro)
@@ -13,5 +13,4 @@
     <xacro:include filename="$(find scout_description)/urdf/camera.xacro"/>         <!-- camera.xacro 추가 -->
     <xacro:include filename="$(find scout_description)/urdf/depth_camera.xacro"/>   <!-- depth_camera 추가 -->
-    <!-- <xacro:include filename="$(find scout_description)/urdf/double_camera.xacro"/>   camera + depth camera 추가 -->
     <xacro:include filename="$(find scout_description)/urdf/gripper.xacro"/>   <!-- gripper 추가 -->
     <!-- Variables -->
